File: Hardware/v1/SunEater.kicad_sch (KiCad schematic)
At the start: 35 parts, among them J1 GPIO, U1 CAT24C256, U2 STM32F103CBTx

Commit message: update to v1
Parts:
- removed U?: TMP100, Package_TO_SOT_SMD:SOT-23-6, symbol Sensor_Temperature:TMP100
- added J?: Conn_02x05_Odd_Even, symbol Connector_Generic:Conn_02x05_Odd_Even
- added J? (x2): Conn_01x02, symbol Connector_Generic:Conn_01x02
- added J?: Conn_01x03, symbol Connector_Generic:Conn_01x03
- added JP?: SolderJumper_2_Open, symbol Jumper:SolderJumper_2_Open
- added R? (x2): R_US, symbol Device:R_US
- added U? (x2): INA700, symbol SunEater:INA700
- added U?: HDC2080, Package_SON:Texas_PWSON-N6, symbol Sensor_Humidity:HDC2080
Connections:
- net +3V3: now also J?.1 (Pin_1), R?.1, R?.1, U?.5 (VDD), U?.B2 (A0), U?.C1 (VS), U?.C1 (VS)
- net CANH: now also J?.2 (Pin_2)
- net CANL: now also J?.3 (Pin_3)
- net GND: now also J?.1 (Pin_1), J?.2 (Pin_2), J?.2 (Pin_2), J?.3 (Pin_3), J?.5 (Pin_5), J?.9 (Pin_9), U?.2 (GND), U?.3 (ADDR), U?.B1 (GND), U?.B1 (GND), U?.B2 (A0)
- net GPIO14/TXD0: now also U2.13 (PA3)
- net GPIO15/RXD0: now also U2.12 (PA2)
- net GPIO23: now also J?.10 (Pin_10), JP?.2 (B)
- net SDA2: now reaches R?.1
- net SDA2: now also U2.22 (PB11), U?.1 (SDA), U?.B3 (SDA), U?.B3 (SDA)
- net SCL2: now reaches R?.1
- net SCL2: now also U2.21 (PB10), U?.6 (SCL), U?.C3 (SCL), U?.C3 (SCL)
- net INT/TMP_SENSOR: now reaches U2.30 (PA9)
- net INT/TMP_SENSOR: now also U?.4 (DRDY)
- net INT/PNL_SENS: now reaches U2.31 (PA10)
- net INT/PNL_SENS: now also R?.2, U?.C2 (ALERT)
- net INT/BAT_SENS: now reaches U2.32 (PA11)
- net INT/BAT_SENS: now also R?.2, U?.C2 (ALERT)
- net SWDIO/TMS: now reaches U2.34 (PA13)
- net SWDIO/TMS: now also J?.2 (Pin_2)
- net SWCLK/TCK: now reaches U2.37 (PA14)
- net SWCLK/TCK: now also J?.4 (Pin_4)
- net TDI: now reaches U2.38 (PA15)
- net TDI: now also J?.8 (Pin_8)
- net SWO/TDO: now reaches U2.39 (PB3)
- net SWO/TDO: now also J?.6 (Pin_6)
- net TRST: now reaches U2.40 (PB4)
- net TRST: now also JP?.1 (A)
- new net: J?.1 (Pin_1), U?.A3 (IN+) (x2)
Other:
- moved on the sheet: R?
